File: pcb/adapter_pcb/adapter_pcb.kicad_pcb (KiCad board)
At the start: 2 copper layers, 50.8 x 50.8 mm, 12 parts, among them J1_MB1 Conn_01x16_Pin, J1_breakout1 Conn_02x10_Counter_Clockwise, J2_MB1 Conn_01x16_Pin, J3 Conn_01x16_Pin, J4 Conn_01x10_Male, J4_breakout1 Conn_01x10_Male, J5 Conn_01x16_Pin, J8_breakout1 Conn_02x10_Counter_Clockwise

Commit message: updated adapter-pcb + gerber zip files(need yichen to review)
Parts:
- removed H1, H6, H7, H8: MountingHole_Pad, MountingHole:MountingHole_3.2mm_M3_Pad_Via
- removed J1_breakout1, J8_breakout1: Conn_02x10_Counter_Clockwise, Connector_PinHeader_2.54mm:PinHeader_2x10_P2.54mm_Vertical
- removed J4: Conn_01x10_Male, Connector_PinHeader_2.54mm:PinHeader_1x10_P2.54mm_Vertical
- removed J4_breakout1: Conn_01x10_Male, external-libs:wirebondarray-dteal
- added J1: Conn_01x10_Socket, external-libs:wirebondarray-dteal, F.Cu at (116.5, 91.5)
- added J3_breakoutL1: Conn_01x20_Socket, external-libs:wirebondarray-1x20-emtan, F.Cu at (110.0, 71.0)
- added J5_breakoutR1: Conn_01x20_Socket, external-libs:wirebondarray-1x20-emtan, F.Cu at (132.0, 71.0)
- added REF**: MountingHole_3.2mm_M3_Pad_Via, MountingHole:MountingHole_3.2mm_M3_Pad_Via, F.Cu at (131.3, 60.5)
- added REF**: MountingHole_3.2mm_M3_Pad_Via, MountingHole:MountingHole_3.2mm_M3_Pad_Via, F.Cu at (111.3, 100.5)
- added REF**: MountingHole_3.2mm_M3_Pad_Via, MountingHole:MountingHole_3.2mm_M3_Pad_Via, F.Cu at (111.3, 60.5)
- added REF**: MountingHole_3.2mm_M3_Pad_Via, MountingHole:MountingHole_3.2mm_M3_Pad_Via, F.Cu at (131.3, 100.5)
- moved J2_MB1 38.5 mm to (141.5, 61.5)
- moved J3 38.4 mm to (101.0, 61.5)
- moved J1_MB1 1.00 mm to (98.3, 61.5)
- moved J5 1.00 mm to (144.0, 61.5)
Routing:
- net Net-(J1-Pin_1): track 0.00 -> 106.6 mm
- net GND: track 148.6 -> 62.1 mm
- net SDA3: track 47.4 -> 14.8 mm
- net +3.3V: track 42.0 -> 11.8 mm
- net +250V: track 42.0 -> 12.4 mm
- net SCL4: track 42.0 -> 12.9 mm
- net SDA4: track 42.2 -> 13.5 mm
- net SCL3: track 42.8 -> 14.1 mm
- net SCL1: track 46.3 -> 18.8 mm
- net SDA2: track 44.1 -> 17.2 mm
- net SDA1: track 44.6 -> 20.3 mm
- net Net-(J2_MB1-Pin_16): track 0.00 -> 20.4 mm
- net Net-(J2_MB1-Pin_15): track 0.00 -> 18.8 mm
- net Net-(J2_MB1-Pin_14): track 0.00 -> 17.2 mm
- net Net-(J1_MB1-Pin_2): track 0.00 -> 15.8 mm
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- added copper zone on B.Cu, net GND
- added copper zone on F.Cu, net GND
Other:
- outline, holes or cut-outs redrawn
