File: pcb/adapter_pcb/adapter_pcb.kicad_sch (KiCad schematic)
At the start: 8 parts, among them J1_MB1 Conn_01x16_Pin, J1_breakout1 Conn_02x10_Counter_Clockwise, J2_MB1 Conn_01x16_Pin, J3 Conn_01x16_Pin, J4 Conn_01x10_Male, J4_breakout1 Conn_01x10_Male, J5 Conn_01x16_Pin, J8_breakout1 Conn_02x10_Counter_Clockwise

Commit message: updated adapter-pcb + gerber zip files(need yichen to review)
Parts:
- removed J1_breakout1, J8_breakout1: Conn_02x10_Counter_Clockwise, Connector_PinHeader_2.54mm:PinHeader_2x10_P2.54mm_Vertical, symbol Connector_Generic:Conn_02x10_Odd_Even
- removed J4: Conn_01x10_Male, Connector_PinHeader_2.54mm:PinHeader_1x10_P2.54mm_Vertical, symbol Connector:Conn_01x10_Male
- removed J4_breakout1: Conn_01x10_Male, external-libs:wirebondarray-dteal, symbol Connector:Conn_01x10_Male
- added J1: Conn_01x10_Socket, external-libs:wirebondarray-dteal, symbol Connector:Conn_01x10_Socket
- added J3_breakoutL1, J5_breakoutR1: Conn_01x20_Socket, external-libs:wirebondarray-1x20-emtan, symbol Connector:Conn_01x20_Socket
Connections:
- net +250V: now also J3_breakoutL1.6 (Pin_6)
- net +3.3V: now also J3_breakoutL1.7 (Pin_7)
- net GND: now also J3_breakoutL1.1 (Pin_1), J3_breakoutL1.8 (Pin_8)
- net SCL1: now also J3_breakoutL1.15 (Pin_15)
- net SCL2: now also J3_breakoutL1.13 (Pin_13)
- net SCL3: now also J3_breakoutL1.11 (Pin_11)
- net SCL4: now also J3_breakoutL1.9 (Pin_9)
- net SDA1: now also J3_breakoutL1.16 (Pin_16)
- net SDA2: now also J3_breakoutL1.14 (Pin_14)
- net SDA3: now also J3_breakoutL1.12 (Pin_12)
- net SDA4: now also J3_breakoutL1.10 (Pin_10)
- net at J2_MB1.1 (Pin_1), J5.1 (Pin_1): now also J1.1 (Pin_1), J5_breakoutR1.1 (Pin_1)
- net at J2_MB1.10 (Pin_10), J5.10 (Pin_10): now also J5_breakoutR1.10 (Pin_10)
- net at J2_MB1.11 (Pin_11), J5.11 (Pin_11): now also J5_breakoutR1.11 (Pin_11)
- net at J2_MB1.12 (Pin_12), J5.12 (Pin_12): now also J5_breakoutR1.12 (Pin_12)
- net at J2_MB1.13 (Pin_13), J5.13 (Pin_13): now also J5_breakoutR1.13 (Pin_13)
- net at J2_MB1.14 (Pin_14), J5.14 (Pin_14): now also J5_breakoutR1.14 (Pin_14)
- net at J2_MB1.15 (Pin_15), J5.15 (Pin_15): now also J5_breakoutR1.15 (Pin_15)
- net at J2_MB1.16 (Pin_16), J5.16 (Pin_16): now also J5_breakoutR1.16 (Pin_16)
- net at J2_MB1.2 (Pin_2), J5.2 (Pin_2): now also J5_breakoutR1.2 (Pin_2)
- net at J2_MB1.3 (Pin_3), J5.3 (Pin_3): now also J5_breakoutR1.3 (Pin_3)
- net at J2_MB1.4 (Pin_4), J5.4 (Pin_4): now also J5_breakoutR1.4 (Pin_4)
- net at J2_MB1.5 (Pin_5), J5.5 (Pin_5): now also J5_breakoutR1.5 (Pin_5)
- net at J2_MB1.6 (Pin_6), J5.6 (Pin_6): now also J5_breakoutR1.6 (Pin_6)
- net at J2_MB1.7 (Pin_7), J5.7 (Pin_7): now also J5_breakoutR1.7 (Pin_7)
- net at J2_MB1.8 (Pin_8), J5.8 (Pin_8): now also J5_breakoutR1.8 (Pin_8)
- net at J2_MB1.9 (Pin_9), J5.9 (Pin_9): now also J5_breakoutR1.9 (Pin_9)
- net at J1_MB1.2 (Pin_2), J3.2 (Pin_2): now also J3_breakoutL1.2 (Pin_2)
- net at J1_MB1.3 (Pin_3), J3.3 (Pin_3): now also J3_breakoutL1.3 (Pin_3)
- net at J1_MB1.4 (Pin_4), J3.4 (Pin_4): now also J3_breakoutL1.4 (Pin_4)
- net at J1_MB1.5 (Pin_5), J3.5 (Pin_5): now also J3_breakoutL1.5 (Pin_5)
Other:
- moved on the sheet: J2_MB1
